File: pcb/one-inch-laserdriver.kicad_sch (KiCad schematic)
At the start: 1 part

Commit message: almost done v1
Parts:
- removed N1: V20220506, SquantorLabels:Label_Generic, symbol SquantorLabels:VYYYYMMDD
- added C1, C4, C5: 0.1uF, Capacitor_SMD:C_0603_1608Metric, symbol Device:C
- added C2, C3: 10uF, Capacitor_SMD:C_0603_1608Metric, symbol Device:C
- added D1, D2, D3: LED, LED_SMD:LED_0603_1608Metric, symbol Device:LED
- added D4: D_Schottky, Diode_SMD:D_SOD-123, symbol Device:D_Schottky
- added J1, J2: Conn_Coaxial, Connector_Coaxial:MMCX_Molex_73415-1471_Vertical, symbol Connector:Conn_Coaxial
- added J3: Power, Connector_PinHeader_2.54mm:PinHeader_1x02_P2.54mm_Vertical, symbol Connector_Generic:Conn_01x02
- added LD1: D_Laser_Photo_NType, OptoDevice:LaserDiode_TO18-D5.6-3, symbol Device:D_Laser_Photo_NType
- added R1, R4, R5, R6: 1k, Resistor_SMD:R_0603_1608Metric, symbol Device:R
- added R2, R3: 3.3, Resistor_SMD:R_0603_1608Metric, symbol Device:R
- added RV1: 1k, Potentiometer_SMD:Potentiometer_Bourns_3314G_Vertical, symbol Device:R_Potentiometer_Trim
- added U1: iC-HK, Package_SO:SO-8_3.9x4.9mm_P1.27mm, symbol ichaus:ic-HK
- added U2: LM1117MP-5.0, Package_TO_SOT_SMD:SOT-223-3_TabPin2, symbol Regulator_Linear:LM1117MP-5.0
Connections:
- new net: C1.1, C2.1, D4.1 (K), U2.3 (VI)
- new net: R6.2, RV1.2
- new net: J2.1 (In), R5.1, U1.5 (EN2)
- new net: D3.2 (A), R5.2
- new net: J1.1 (In), R4.1, U1.1 (EN1)
- new net: R2.2, U1.2 (AGND1)
- new net: LD1.1, U1.3 (LDK)
- new net: R3.1, U1.4 (AGND2)
- new net: R6.1, U1.8 (CI)
- new net: D1.2 (A), R1.2
- new net: D2.2 (A), R4.2
- new net: D4.2 (A), J3.2 (Pin_2)
- new net +5V: C3.1, C4.1, C5.1, LD1.2, R1.1, RV1.3, U1.7 (VDD), U2.2 (VO)
- new net GND: C1.2, C2.2, C3.2, C4.2, C5.2, D1.1 (K), D2.1 (K), D3.1 (K), J1.2 (Ext), J2.2 (Ext), J3.1 (Pin_1), R2.1, R3.2, RV1.1, U1.6 (GND), U2.1 (GND)
Other:
- note removed: "Labels"
- note removed: "Mechanical"
- note removed: "Powersupply stuff"

Commit message: bias tee
Parts:
- removed D3: LED, LED_SMD:LED_0603_1608Metric, symbol Device:LED
- removed U2: LM1117MP-5.0, Package_TO_SOT_SMD:SOT-223-3_TabPin2, symbol Regulator_Linear:LM1117MP-5.0
- added C6: 0.1uF, Capacitor_SMD:C_0603_1608Metric, symbol Device:C
- added L1: 22uH, symbol Device:L
- added U3: HT75xx-1-SOT89, Package_TO_SOT_SMD:SOT-89-3, symbol Regulator_Linear:HT75xx-1-SOT89
- R5: value 1k -> 47
Connections:
- net +5V: now also U3.3 (VOUT)
- net GND: now also U3.1 (GND)
- net at C1.1, C2.1, D4.1 (K): now also U3.2 (VIN)
- net at R5.2: now also LD1.1
- net at U1.3 (LDK): now also L1.2; no longer LD1.1
- new net: C6.1, J2.1 (In)
- new net: C6.2, L1.1, R5.1
- now unconnected: U1.5 (EN2)
Other:
- moved on the sheet: C4, C5, D2, J1, J2, LD1, R2, R3, R4, R6, RV1, U1

Commit message: ic-HKb version done
Parts:
- removed J1: Conn_Coaxial, Connector_Coaxial:MMCX_Molex_73415-1471_Vertical, symbol Connector:Conn_Coaxial
- added C7: 0.1uF, Capacitor_SMD:C_0402_1005Metric, symbol Device:C
- added C8: 10uF, Capacitor_SMD:C_0603_1608Metric, symbol Device:C
- added JP1: SolderJumper_3_Bridged12, Jumper:SolderJumper-3_P1.3mm_Open_RoundedPad1.0x1.5mm_NumberLabels, symbol Jumper:SolderJumper_3_Bridged12
- added R7: 10, Resistor_SMD:R_0603_1608Metric, symbol Device:R
- added R8: 10k, Resistor_SMD:R_0402_1005Metric, symbol Device:R
- added R9: 47*, Resistor_SMD:R_0402_1005Metric, symbol Device:R
- added TP1: 9V, TestPoint:TestPoint_THTPad_D1.0mm_Drill0.5mm, symbol Connector:TestPoint
- added TP2: 5V, TestPoint:TestPoint_THTPad_D1.0mm_Drill0.5mm, symbol Connector:TestPoint
- added TP3: GND, TestPoint:TestPoint_THTPad_D1.0mm_Drill0.5mm, symbol Connector:TestPoint
- added TP4: LDC, TestPoint:TestPoint_THTPad_D1.0mm_Drill0.5mm, symbol Connector:TestPoint
- added TP5: CI, TestPoint:TestPoint_THTPad_D1.0mm_Drill0.5mm, symbol Connector:TestPoint
- added TP6: Hole, TestPoint:TestPoint_THTPad_D1.0mm_Drill0.5mm, symbol Connector:TestPoint
- added U2: HT7590-3, Package_TO_SOT_SMD:SOT-23-5, symbol Regulator_Linear:HT75xx-1-SOT89
- C1, C4, C5, C6: footprint Capacitor_SMD:C_0603_1608Metric -> Capacitor_SMD:C_0402_1005Metric; LCSC (none) -> C307331
- C2, C3: LCSC (none) -> C96446
- D1, D2: LCSC (none) -> C72043
- J2: LCSC (none) -> C5137198
- L1: footprint (none) -> Inductor_SMD:L_Sunlord_SWPA4018S; LCSC (none) -> C83443
- R1, R6: footprint Resistor_SMD:R_0603_1608Metric -> Resistor_SMD:R_0402_1005Metric; LCSC (none) -> C11702
- R2, R3: value 3.3 -> 1; LCSC (none) -> C22936
- R4: value 1k -> 10k; footprint Resistor_SMD:R_0603_1608Metric -> Resistor_SMD:R_0402_1005Metric; LCSC (none) -> C25744
- R5: footprint Resistor_SMD:R_0603_1608Metric -> Resistor_SMD:R_0402_1005Metric; LCSC (none) -> C25118
- U3: value HT75xx-1-SOT89 -> HT7550-2; footprint Package_TO_SOT_SMD:SOT-89-3 -> Package_TO_SOT_SMD:SOT-23-5; LCSC C16106 -> C81799
Connections:
- net +5V: now also R4.2, TP2.1; no longer C5.1, LD1.2, R1.1
- net GND: now also C7.2, C8.2, R8.1, TP3.1, U2.1 (GND)
- net at C6.1: now also JP1.1 (A); no longer J2.1 (In)
- net at C6.2, L1.1, R5.1: now also R9.2, TP4.1
- net at R4.1, U1.1 (EN1): now also JP1.3 (B)
- net at U1.5 (EN2): now also R8.2
- net at R6.1, U1.8 (CI): now also TP5.1
- net at D1.2 (A), R1.2: now also D2.2 (A)
- net at LD1.3: now also R9.1
- net at C1.1, C2.1, U3.2 (VIN): now also R1.1, C7.1, R7.2, U2.2 (VIN); no longer D4.1 (K)
- new net: J2.1 (In), JP1.2 (C)
- new net: D4.1 (K), R7.1
- new net +9V: C5.1, C8.1, LD1.2, TP1.1, U2.3 (VOUT)
Other:
- note added: "Populate R9 for Type D, R5 for Type A"
- moved on the sheet: D1, D4, J2, J3, R1

Commit message: working. standard design
Parts:
- R1: value 1k -> 2.2k; footprint Resistor_SMD:R_0402_1005Metric -> Resistor_SMD:R_0603_1608Metric; LCSC C11702 -> C4190
- R4, R8: footprint Resistor_SMD:R_0402_1005Metric -> Resistor_SMD:R_0603_1608Metric; LCSC C25744 -> C25804
- R5: now not fitted
- R6: footprint Resistor_SMD:R_0402_1005Metric -> Resistor_SMD:R_0603_1608Metric; LCSC C11702 -> C21190
- R9: value 47* -> 47
Connections:
- net +5V: now also RV1.1; no longer RV1.3
- net GND: now also RV1.3, TP6.1; no longer RV1.1
Other:
- moved on the sheet: RV1
